File: versions/with_inverted_ampl.kicad_pcb (KiCad board)
At the start: 2 copper layers, 50 x 24 mm, 16 parts, among them Q1 2SC3356, Q3 2SC3356

Commit message: asdasd
Parts:
- moved R3 3.73 mm to (47.2, 58.8)
- moved R1 3.22 mm to (42.8, 58.0), turned to -90 degrees
- moved C104 2.67 mm to (37.9, 65.3)
- moved RData1 2.44 mm to (41.0, 62.4)
- moved 5_pins_op_amp1 2.31 mm to (46.5, 62.5)
- moved R6 1.03 mm to (40.2, 58.0), turned to 90 degrees
- moved 8_pin_op_amp1 0.81 mm to (51.7, 64.8)
- moved R2 0.60 mm to (42.8, 65.9)
Routing:
- net Net-(5_pins_op_amp1-VOUT): track 44.6 -> 24.3 mm
- net Net-(5_pins_op_amp1-VDD): track 55.8 -> 43.5 mm
- net Net-(Q1-C): track 10.7 -> 17.5 mm
- net Net-(A1-+5V): track 3.35 -> 0.07 mm
- net Net-(5_pins_op_amp1-VIN-): track 19.6 -> 17.1 mm
