File: diploma_pcb/diploma_pcb.kicad_pcb (KiCad board)
At the start: 2 copper layers, 50 x 24 mm, 21 parts, among them Q1 2SC3356, Q3 2SC3356

Commit message: changes on schematic
Parts:
- R1: value R -> 1K
Changed lines of the file:
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@@
 			)
 		)
-		(property "Value" "R"
+		(property "Value" "1K"
 			(at 0 1.82 0)
 			(layer "F.Fab")

Commit message: PCB values chosen and set
Parts:
- R1: value 1K -> R
Changed lines of the file:
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@@
 			)
 		)
-		(property "Value" "1K"
+		(property "Value" "R"
 			(at 0 1.82 0)
 			(layer "F.Fab")
