File: V2/Pico_PCB/Entry/Entry.kicad_sch (KiCad schematic)
At the start: 24 parts, among them Q2 2n3904

Commit message: Documentation solid V1
Parts:
- removed D1, D2, D3: MBRS1100T3G, MBRS1100T3G:SMB_403A-03_ONS, symbol MBRS1100T3G:MBRS1100T3G
- added D1, D2, D3: D_Schottky, MBRS1100T3G:SMB_403A-03_ONS, symbol Device:D_Schottky
- renumbered OpAmp to OpAmp1, R_LED_B1 to R6, R_LED_G1 to R7, R_LED_R1 to R8
Connections:
- net at C1.1: now also D1.1 (K), D2.2 (A)
- net at C2.1: now also D2.1 (K), D3.2 (A)
- net at C3.1, R1.2: now also D3.1 (K)
- net 5V: no longer names the net of C6.2, PicoW1.40 (VBUS)
- net 5V: now also D1.2 (A)
- net blue: no longer names the net of LED1.6 (A_BLUE), R6.2
- net green: no longer names the net of LED1.4 (A_GREEN), R7.2
- net red: no longer names the net of LED1.2 (A_RED), R8.2
- no-connect marks 1 -> 28
Other:
- note added: "3.3V"
- note added: "5V"
- moved on the sheet: LED1, R6, R7, R8
